Commit message: Add readme

File: resources/robots/mini_cheetah/mini_cheetah.urdf (robot description, URDF)
Before this commit: robot mini_cheetah, 17 links, 16 joints
Links:
- added link world
Joints:
- added joint world_joint: type fixed, parent world, child body, origin xyz=0.0 0.0 0.6 rpy=0.3 0 0
